File: pcb-design/sudi-redox-clone.kicad_sch (KiCad schematic)
At the start: 109 parts, among them J1 SIDE_CON, J2 0.91 OLED, J4 USBC_PWR_ONLY, J5 SIDE_CON, J7 ARMJTAG, J8 BatCon, K1 KEYSW, K10 KEYSW, K11 KEYSW, K12 KEYSW, K13 KEYSW, K14 KEYSW, K15 KEYSW, K16 KEYSW, K17 KEYSW, K18 KEYSW, K2 KEYSW, K3 KEYSW, K4 KEYSW, K5 KEYSW, K6 KEYSW, K7 KEYSW, K8 KEYSW, K9 KEYSW, SW1 RST, U4 AMS1117-3.3, U5 CH340G, U6 TP4056, U7 nRF52832-QFxx, U8 MCP23017_SS, Y5 32MHz

Commit message: add CH340C
Parts:
- removed J4: USBC_PWR_ONLY, Connector_USB:USB_C_Receptacle_GCT_USB4125-xx-x-0190_6P_TopMnt_Horizontal, symbol Connector:USB_C_Receptacle_PowerOnly_6P
- removed U5: CH340G, Package_SO:SOIC-16_3.9x9.9mm_P1.27mm, symbol Interface_USB:CH340G
- added P1: USB_C_Plug_USB2.0, Connector_USB:USB_C_Receptacle_GCT_USB4105-xx-A_16P_TopMnt_Horizontal, symbol Connector:USB_C_Plug_USB2.0
- added U5: CH340C, Package_SO:SOIC-16_3.9x9.9mm_P1.27mm, symbol Interface_USB:CH340C
Connections:
- net +3.3V: now also U5.16 (VCC), U5.4 (V3)
- net GND: now also P1.A1 (GND), P1.A12 (GND), P1.B1 (GND), P1.B12 (GND), P1.S1 (SHIELD), U5.1 (GND)
- net at R3.1: now also P1.A5 (CC)
- net at R4.1: now also P1.B5 (VCONN)
- net at FB1.1: now also P1.A4 (VBUS), P1.A9 (VBUS), P1.B4 (VBUS), P1.B9 (VBUS)
- net USART1_RX renamed RX
- net RX: now also U5.2 (TXD)
- net USART1_TX renamed TX
- net TX: now also U5.3 (RXD)
- new net: P1.A6 (D+), U5.5 (UD+)
- new net: P1.A7 (D-), U5.6 (UD-)
- no-connect marks 23 -> 31
Other:
- note added: "ADD USB C Backup with usb serial converter"
- note removed: "ADD USB B Backup"
- moved on the sheet: D1, D10, D11, D12, D13, D14, D15, D16, D17, D18, D19, D2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

Commit message: [11-01-1954] add test point into NRF
Parts:
- removed J7: ARMJTAG, Connector_PinHeader_2.54mm:PinHeader_2x05_P2.54mm_Horizontal, symbol Connector:Conn_ARM_JTAG_SWD_10
- added J3: SWD_JLINK, Connector_PinHeader_2.54mm:PinHeader_1x04_P2.54mm_Horizontal, symbol Connector:Conn_01x04_Socket
- added TP1, TP10, TP11, TP12, TP13, TP14, TP15, TP16, TP17, TP18, TP2, TP3, TP4, TP5, TP6, TP7, TP8, TP9: TestPoint, TestPoint:TestPoint_Pad_D1.0mm, symbol Connector:TestPoint
Connections:
- net +3.3V: now also J3.4 (Pin_4)
- net GND: now also J3.1 (Pin_1)
- net SWCLK: now also J3.2 (Pin_2)
- net SWDIO: now also J3.3 (Pin_3)
- net P0.00/XL1: now reaches U7.2 (P0.00/XL1)
- net P0.00/XL1: now also TP13.1
- net P0.19: now reaches U7.22 (P0.19)
- net P0.19: now also TP1.1
- net P0.20: now reaches U7.23 (P0.20)
- net P0.20: now also TP3.1
- net P0.22: now reaches U7.27 (P0.22)
- net P0.22: now also TP2.1
- net P0.23: now reaches U7.28 (P0.23)
- net P0.23: now also TP4.1
- net P0.24: now reaches U7.29 (P0.24)
- net P0.24: now also TP5.1
- net P0.01/XL2: now reaches U7.3 (P0.01/XL2)
- net P0.01/XL2: now also TP14.1
- net P0.25: now reaches U7.37 (P0.25)
- net P0.25: now also TP6.1
- net P0.26: now reaches U7.38 (P0.26)
- net P0.26: now also TP7.1
- net P0.27: now reaches U7.39 (P0.27)
- net P0.27: now also TP8.1
- net P0.02/AIN0: now reaches U7.4 (P0.02/AIN0)
- net P0.02/AIN0: now also TP15.1
- net P0.28/AIN4: now reaches U7.40 (P0.28/AIN4)
- net P0.28/AIN4: now also TP9.1
- net P0.29/AIN5: now reaches U7.41 (P0.29/AIN5)
- net P0.29/AIN5: now also TP10.1
- net P0.30/AIN6: now reaches U7.42 (P0.30/AIN6)
- net P0.30/AIN6: now also TP11.1
- net P0.31/AIN7: now reaches U7.43 (P0.31/AIN7)
- net P0.31/AIN7: now also TP12.1
- net P0.03/AIN1: now reaches U7.5 (P0.03/AIN1)
- net P0.03/AIN1: now also TP16.1
- net P0.04/AIN2: now reaches U7.6 (P0.04/AIN2)
- net P0.04/AIN2: now also TP17.1
- net P0.05/AIN3: now reaches U7.7 (P0.05/AIN3)
- net P0.05/AIN3: now also TP18.1
- no-connect marks 31 -> 28
Other:
- note added: "Currently Excluded"
- note removed: "TODO Change JTAG Connector As Jlink SWD Pinout"
- note removed: "V2 TODO make it wireless with NRF51822 add BMS to System (TP4056) make receiver and transmitter with NRF use LUFA with ATMega8 for usb receiver / RECEIVER SCH https://www.fourwalledcubicle.com/files/LUFA/Doc/120219/html/_page__a_v_r8_support.html https://developer.nordicsemi.com/nRF5_SDK/nRF51_SDK_v4.x.x/doc/html/group__ble__sdk__app__hids__keyboard.html"
- moved on the sheet: C1, C4, D4, J8, R6, R7, U6
