File: pcb-design/Receiver.kicad_sch (KiCad schematic)
At the start: 29 parts, among them J6 USB_A, J9 ARM_JTAG, SW2 SW_Push, U1 ATmega32A-A, U2 nRF51x22-QFxx, U3 AMS1117-3.3, Y1 16MHz, Y3 16MHz

Commit message: [minggu 7 juli 8:55] cleaning schematic layout
Parts:
- removed U1: ATmega32A-A, Package_QFP:TQFP-44_10x10mm_P0.8mm, symbol MCU_Microchip_ATmega:ATmega32A-A
- added C10: 1uF, symbol Device:C
- added C23, C7: 100nF, symbol Device:C
- added J9: AVR-ISP-6, symbol Connector:AVR-ISP-6
- added R8: 1K, Resistor_SMD:R_1206_3216Metric, symbol Device:R_US
- added U2: ATmega8U2-A, Package_QFP:TQFP-32_7x7mm_P0.8mm, symbol MCU_Microchip_ATmega:ATmega8U2-A
- C5: renamed from C28; value 12pF -> 22pF
- C6: renamed from C29; value 12pF -> 22pF
- SW2: value SW_Push -> RCV_RST
- Y1: renamed from Y3; value 16MHz -> 8MHz
- renumbered C31 to C22, C5 to C24, C6 to C25, C7 to C26, C9 to C27, C10 to C28, C22 to C29, C23 to C30, C24 to C31, C25 to C32, C26 to C33, C27 to C34, C30 to C9, J9 to J10, R8 to R9, U3 to U1, U2 to U3, Y1 to Y3
Connections:
- net +3.3V: now also C23.1, U2.31 (UVCC), U2.32 (AVCC), U2.4 (VCC)
- net +5V: now also J9.2 (VCC), R8.2
- net GND: now also SW2.1, C10.2, C23.2, C7.2, J9.6 (GND), U2.28 (UGND), U2.3 (GND)
- net RCV_USART1_RX: now also U2.8 (PD2)
- net RCV_USART1_TX: now also U2.9 (PD3)
- net at C6.2, Y1.2: now also U2.2 (PC0/XTAL2)
- net at C5.2, Y1.1: now also U2.1 (XTAL1)
- net at J6.2 (D-): now also U2.30 (D-)
- net at J6.3 (D+): now also U2.29 (D+)
- net RCV_RST: now reaches SW2.2
- net RCV_RST: now also C7.1, J9.5 (~{RST}), R8.1, U2.24 (PC1/~{RESET})
- new net: C10.1, U2.27 (UCAP)
- new net RCV_MISO: J9.1 (MISO), U2.17 (PB3)
- new net RCV_MOSI: J9.4 (MOSI), U2.16 (PB2)
- new net RCV_SCK: J9.3 (SCK), U2.15 (PB1)
Other:
- note added: "Maximum Frequency - 8 MHz at 2.7V - Industrial range - 16 MHz at 4.5V - Industrial range"
- note added: "References: ATmega8U2 ATmega16U2 ATmega32U2 Datasheet"
- moved on the sheet: AE2, C22, C24, C25, C26, C27, C28, C29, C30, C31, C32, C33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

Commit message: [minggu 7 juli 12:12] create pcb cut profile
Parts:
- removed Y1: 8MHz, symbol Device:Crystal
- added Y4: 8MHz, Crystal:Crystal_HC50_Vertical, symbol Device:Crystal
- C10, C22, C23, C24, C25, C26, C27, C28, C29, C30, C31, C32, C33, C34, C5, C6, C7, C9: footprint (none) -> Capacitor_SMD:C_0805_2012Metric_Pad1.18x1.45mm_HandSolder
- FB2, L4, L5, L6: footprint (none) -> Inductor_SMD:L_0603_1608Metric_Pad1.05x0.95mm_HandSolder
- J6: footprint Connector_USB:USB_A_CONNFLY_DS1095-WNR0 -> Connector_USB:USB_A_CNCTech_1001-011-01101_Horizontal
- J9: footprint (none) -> Connector_PinHeader_2.54mm:PinHeader_2x05_P2.54mm_Vertical
- SW2: footprint (none) -> Button_Switch_SMD:SW_Push_1P1T_NO_6x6mm_H9.5mm
- Y3: footprint (none) -> Crystal:Crystal_HC50_Vertical
Connections:
- net at C6.2, U2.2 (PC0/XTAL2): now also Y4.2
- net at C5.2, U2.1 (XTAL1): now also Y4.1
Changed lines of the file:
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@@
 	)
 	(junction
-		(at 43.18 40.64)
-		(diameter 0)
-		(color 0 0 0 0)
-	)
-	(junction
 		(at 163.83 67.31)
 		(diameter 0)
@@
 	)
 	(junction
-		(at 43.18 48.26)
-		(diameter 0)
-		(color 0 0 0 0)
-	)
-	(junction
 		(at 193.04 90.17)
 		(diameter 0)
@@
 	)
 	(junction
+		(at 41.91 40.64)
+		(diameter 0)
+		(color 0 0 0 0)
+	)
+	(junction
 		(at 33.02 92.71)
 		(diameter 0)
@@
 	)
 	(junction
+		(at 41.91 48.26)
+		(diameter 0)
+		(color 0 0 0 0)
+	)
+	(junction
 		(at 81.28 46.99)
 		(diameter 0)
@@
 	(wire
 		(pts
-			(xy 46.99 48.26) (xy 43.18 48.26)
-		)
-		(stroke
-			(width 0)
-			(type default)
-		)
-	)
-	(wire
-		(pts
 			(xy 186.69 90.17) (xy 193.04 90.17)
 		)
@@
 	(wire
 		(pts
+			(xy 41.91 48.26) (xy 46.99 48.26)
+		)
+		(stroke
+			(width 0)
+			(type default)
+		)
+	)
+	(wire
+		(pts
 			(xy 101.6 63.5) (xy 118.11 63.5)
 		)
@@
 	(wire
 		(pts
+			(xy 41.91 40.64) (xy 46.99 40.64)
+		)
+		(stroke
+			(width 0)
+			(type default)
+		)
+	)
+	(wire
+		(pts
 			(xy 193.04 49.53) (xy 193.04 50.8)
 		)
@@
 	(wire
 		(pts
-			(xy 36.83 48.26) (xy 43.18 48.26)
+			(xy 36.83 48.26) (xy 41.91 48.26)
 		)
 		(stroke
@@
 	(wire
 		(pts
-			(xy 31.75 40.64) (xy 43.18 40.64)
+			(xy 31.75 40.64) (xy 41.91 40.64)
 		)
 		(stroke
@@
 	(wire
 		(pts
-			(xy 43.18 40.64) (xy 46.99 40.64)
-		)
-		(stroke
-			(width 0)
-			(type default)
-		)
-	)
-	(wire
-		(pts
 			(xy 74.93 170.18) (xy 74.93 168.91)
 		)
@@
 			)
 		)
-		(property "Footprint" ""
+		(property "Footprint" "Capacitor_SMD:C_0805_2012Metric_Pad1.18x1.45mm_HandSolder"
 			(at 180.6448 92.71 0)
 			(effects
@@
 			)
 		)
-		(property "Footprint" ""
+		(property "Footprint" "Inductor_SMD:L_0603_1608Metric_Pad1.05x0.95mm_HandSolder"
 			(at 154.94 67.31 0)
 			(effects
@@
 			)
 		)
-		(property "Footprint" ""
+		(property "Footprint" "Capacitor_SMD:C_0805_2012Metric_Pad1.18x1.45mm_HandSolder"
 			(at 199.0852 46.99 0)
 			(effects
@@
 			)
 		)
-		(property "Footprint" ""
+		(property "Footprint" "Capacitor_SMD:C_0805_2012Metric_Pad1.18x1.45mm_HandSolder"
 			(at 146.3548 78.74 0)
 			(effects
@@
 			)
 		)
-		(property "Footprint" ""
+		(property "Footprint" "Capacitor_SMD:C_0805_2012Metric_Pad1.18x1.45mm_HandSolder"
 			(at 37.7952 50.8 0)
 			(effects
@@
 			)
 		)
-		(property "Footprint" ""
+		(property "Footprint" "Capacitor_SMD:C_0805_2012Metric_Pad1.18x1.45mm_HandSolder"
 			(at 187.6552 92.71 0)
 			(effects
@@
 			)
 		)
-		(property "Footprint" ""
+		(property "Footprint" "Capacitor_SMD:C_0805_2012Metric_Pad1.18x1.45mm_HandSolder"
 			(at 30.7848 50.8 0)
 			(effects
@@
 			)
 		)
-		(property "Footprint" ""
+		(property "Footprint" "Capacitor_SMD:C_0805_2012Metric_Pad1.18x1.45mm_HandSolder"
 			(at 244.8052 36.83 0)
 			(effects
@@
 			)
 		)
-		(property "Footprint" ""
+		(property "Footprint" "Inductor_SMD:L_0603_1608Metric_Pad1.05x0.95mm_HandSolder"
 			(at 180.34 60.96 0)
 			(effects
@@
 			)
 		)
-		(property "Footprint" ""
+		(property "Footprint" "Capacitor_SMD:C_0805_2012Metric_Pad1.18x1.45mm_HandSolder"
 			(at 237.1852 36.83 0)
 			(effects
@@
 			)
 		)
-		(property "Footprint" ""
+		(property "Footprint" "Capacitor_SMD:C_0805_2012Metric_Pad1.18x1.45mm_HandSolder"
 			(at 252.4252 36.83 0)
 			(effects
@@
 			)
 		)
-		(property "Footprint" "Connector_USB:USB_A_CONNFLY_DS1095-WNR0"
+		(property "Footprint" "Connector_USB:USB_A_CNCTech_1001-011-01101_Horizontal"
 			(at 36.83 82.55 0)
 			(effects
@@
 			)
 		)
-		(property "Footprint" ""
+		(property "Footprint" "Inductor_SMD:L_0603_1608Metric_Pad1.05x0.95mm_HandSolder"
 			(at 45.72 77.978 90)
 			(effects
@@
 			)
 		)
-		(property "Footprint" ""
+		(property "Footprint" "Button_Switch_SMD:SW_Push_1P1T_NO_6x6mm_H9.5mm"
 			(at 40.64 27.94 0)
 			(effects
@@
 			)
 		)
-		(property "Footprint" ""
+		(property "Footprint" "Capacitor_SMD:C_0805_2012Metric_Pad1.18x1.45mm_HandSolder"
 			(at 179.3748 34.29 0)
 			(effects
@@
 			)
 		)
-		(property "Footprint" ""
+		(property "Footprint" "Capacitor_SMD:C_0805_2012Metric_Pad1.18x1.45mm_HandSolder"
 			(at 92.4052 45.72 0)
 			(effects
@@
 			)
 		)
-		(property "Footprint" ""
+		(property "Footprint" "Capacitor_SMD:C_0805_2012Metric_Pad1.18x1.45mm_HandSolder"
 			(at 36.83 24.4348 0)
 			(effects
@@
 	)
 	(symbol
+		(lib_id "Device:Crystal")
+		(at 41.91 44.45 90)
+		(mirror x)
+		(unit 1)
+		(exclude_from_sim no)
+		(in_bom yes)
+		(on_board yes)
+		(dnp no)
+		(property "Reference" "Y4"
+			(at 38.1 43.1799 90)
+			(effects
+				(font
+					(size 1.27 1.27)
+				)
+				(justify left)
+			)
+		)
+		(property "Value" "8MHz"
+			(at 38.1 45.7199 90)
+			(effects
+				(font
+					(size 1.27 1.27)
+				)
+				(justify left)
+			)
+		)
+		(property "Footprint" "Crystal:Crystal_HC50_Vertical"
+			(at 41.91 44.45 0)
+			(effects
+				(font
+					(size 1.27 1.27)
+				)
+				(hide yes)
+			)
+		)
+		(property "Datasheet" "~"
+			(at 41.91 44.45 0)
+			(effects
+				(font
+					(size 1.27 1.27)
+				)
+				(hide yes)
+			)
+		)
+		(property "Description" "Two pin crystal"
+			(at 41.91 44.45 0)
+			(effects
+				(font
+					(size 1.27 1.27)
+				)
+				(hide yes)
+			)
+		)
+		(pin "2"
+		)
+		(pin "1"
+		)
+		(instances
+			(project "sudi-redox-clone"
+				(path "/5bbd2338-13ff-49b0-9f87-5cbfec528c5b/c474124e-34bd-49d8-8819-329d9c2bdf56"
+					(reference "Y4")
+					(unit 1)
+				)
+			)
+		)
+	)
+	(symbol
 		(lib_id "Device:C_Polarized")
 		(at 74.93 173.99 0)
@@
 			)
 		)
-		(property "Footprint" ""
+		(property "Footprint" "Capacitor_SMD:C_0805_2012Metric_Pad1.18x1.45mm_HandSolder"
 			(at 75.8952 177.8 0)
 			(effects
@@
 			)
 		)
-		(property "Footprint" ""
+		(property "Footprint" "Capacitor_SMD:C_0805_2012Metric_Pad1.18x1.45mm_HandSolder"
 			(at 162.8648 78.74 0)
 			(effects
@@
 			)
 		)
-		(property "Footprint" ""
+		(property "Footprint" "Capacitor_SMD:C_0805_2012Metric_Pad1.18x1.45mm_HandSolder"
 			(at 62.5348 88.9 0)
 			(effects
@@
 			)
 		)
-		(property "Footprint" ""
+		(property "Footprint" "Capacitor_SMD:C_0805_2012Metric_Pad1.18x1.45mm_HandSolder"
 			(at 48.5648 177.8 0)
 			(effects
@@
 			)
 		)
-		(property "Footprint" ""
+		(property "Footprint" "Capacitor_SMD:C_0805_2012Metric_Pad1.18x1.45mm_HandSolder"
 			(at 168.91 66.3448 0)
 			(effects
@@
 			)
 		)
-		(property "Footprint" ""
+		(property "Footprint" "Inductor_SMD:L_0603_1608Metric_Pad1.05x0.95mm_HandSolder"
 			(at 180.34 49.53 0)
 			(effects
@@
 	)
 	(symbol
-		(lib_id "Device:Crystal")
-		(at 43.18 44.45 90)
-		(mirror x)
-		(unit 1)
-		(exclude_from_sim no)
-		(in_bom yes)
-		(on_board yes)
-		(dnp no)
-		(property "Reference" "Y1"
-			(at 39.37 43.1799 90)
-			(effects
-				(font
-					(size 1.27 1.27)
-				)
-				(justify left)
-			)
-		)
-		(property "Value" "8MHz"
-			(at 39.37 45.7199 90)
-			(effects
-				(font
-					(size 1.27 1.27)
-				)
-				(justify left)
-			)
-		)
-		(property "Footprint" ""
-			(at 43.18 44.45 0)
-			(effects
-				(font
-					(size 1.27 1.27)
-				)
-				(hide yes)
-			)
-		)
-		(property "Datasheet" "~"
-			(at 43.18 44.45 0)
-			(effects
-				(font
-					(size 1.27 1.27)
-				)
-				(hide yes)
-			)
-		)
-		(property "Description" "Two pin crystal"
-			(at 43.18 44.45 0)
-			(effects
-				(font
-					(size 1.27 1.27)
-				)
-				(hide yes)
-			)
-		)
-		(pin "2"
-		)
-		(pin "1"
-		)
-		(instances
-			(project "sudi-redox-clone"
-				(path "/5bbd2338-13ff-49b0-9f87-5cbfec528c5b/c474124e-34bd-49d8-8819-329d9c2bdf56"
-					(reference "Y1")
-					(unit 1)
-				)
-			)
-		)
-	)
-	(symbol
 		(lib_id "Device:C")
 		(at 193.04 43.18 0)
@@
 			)
 		)
-		(property "Footprint" ""
+		(property "Footprint" "Capacitor_SMD:C_0805_2012Metric_Pad1.18x1.45mm_HandSolder"
 			(at 192.0748 46.99 0)
 			(effects
@@
 			)
 		)
-		(property "Footprint" ""
+		(property "Footprint" "Crystal:Crystal_HC50_Vertical"
 			(at 193.04 86.36 0)
 			(effects
@@
 			)
 		)
-		(property "Footprint" ""
+		(property "Footprint" "Connector_PinHeader_2.54mm:PinHeader_2x05_P2.54mm_Vertical"
 			(at 120.65 172.72 90)
 			(effects

Commit message: [minggu 7 juli 19:32] finish PCB Layout
Parts:
- R8, R9: footprint Resistor_SMD:R_1206_3216Metric -> Resistor_SMD:R_0805_2012Metric_Pad1.20x1.40mm_HandSolder
Changed lines of the file:
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@@
 			)
 		)
-		(property "Footprint" "Resistor_SMD:R_1206_3216Metric"
+		(property "Footprint" "Resistor_SMD:R_0805_2012Metric_Pad1.20x1.40mm_HandSolder"
 			(at 138.684 162.306 90)
 			(effects
@@
 			)
 		)
-		(property "Footprint" "Resistor_SMD:R_1206_3216Metric"
+		(property "Footprint" "Resistor_SMD:R_0805_2012Metric_Pad1.20x1.40mm_HandSolder"
 			(at 195.834 121.666 90)
 			(effects

Commit message: [16-11-1807] change chargin mechanism
Parts:
- renumbered J9 to J7, J10 to J8, Y4 to Y2
